File: schema/KiCad/TeraCom/TeraCom.kicad_pcb (KiCad board)
At the start: 2 copper layers, 12 parts, among them K1 G5LE-1, K2 G5LE-1, K3 G5LE-1, K5 G5LE-1, U1 ESP32-C6-DevKitM-1, U2 PC817, U3 PC817, U4 PC817, U5 PC817, U6 DS18S20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

Commit message: v0.3
Parts:
- added C1: C_Polarized_Small_US, Capacitor_THT:CP_Radial_D7.5mm_P2.50mm, F.Cu at (36.7, 161.4)
- added C2: C_Polarized_Small_US, Capacitor_THT:CP_Radial_D7.5mm_P2.50mm, F.Cu at (36.7, 170.5)
- added D11: 1N4007, Diode_THT:D_DO-41_SOD81_P10.16mm_Horizontal, F.Cu at (44.4, 159.1)
- added U9: LM7805_TO220, Package_TO_SOT_THT:TO-220-3_Vertical, F.Cu at (45.7, 165.1)
Connections:
- net +12V renamed POWER_RELAY_CARD
- net /Relay_Input3 renamed Relay_Input3
- net /relays/Relay_Input3 renamed Relay_INPUT3
- U1 pad 21: unconnected-(U1-GPIO15/JTAG-Pad21) -> Net-(U1-GPIO15/JTAG)
- U1 pad 22: /Relay_Input2 -> Relay_INPUT2
- U1 pad 23: unconnected-(U1-GPIO19-Pad23) -> Net-(U1-GPIO19)
- U1 pad 25: unconnected-(U1-GPIO21-Pad25) -> Net-(U1-GPIO21)
- U1 pad 28: /Relay_Input1 -> Relay_INPUT1
- U1 pad 29: /Relay_Input4 -> Relay_INPUT4
- U2 pad 2: /relays/Relay_Input1 -> Relay_INPUT1
- U2 pad 3: GND -> GND_RELAY_CARD
- U3 pad 2: /relays/Relay_Input2 -> Relay_INPUT2
- U3 pad 3: GND -> GND_RELAY_CARD
- U4 pad 3: GND -> GND_RELAY_CARD
- U5 pad 2: /relays/Relay_Input4 -> Relay_INPUT4
- U5 pad 3: GND -> GND_RELAY_CARD
- U6 pad 1: unconnected-(U6-GND-Pad1) -> GND_RELAY_CARD
- U6 pad 3: unconnected-(U6-V_{DD}-Pad3) -> +5V
- U7 pad 1: unconnected-(U7-GND-Pad1) -> GND_RELAY_CARD
- U7 pad 3: unconnected-(U7-V_{DD}-Pad3) -> +5V
- U8 pad 1: unconnected-(U8-VDD-Pad1) -> +5V
- U8 pad 4: unconnected-(U8-GND-Pad4) -> GND_RELAY_CARD
