File: schema/KiCad/TeraCom/TeraCom.kicad_sch (KiCad schematic)
At the start: 4 parts, among them U1 ESP32-C6-DevKitM-1, U6 DS18S20, U7 DS18S20, U8 DHT11

Commit message: v0.3
Parts:
- added C1, C2: C_Polarized_Small_US, Capacitor_THT:CP_Radial_D7.5mm_P2.50mm, symbol Device:C_Polarized_Small_US
- added D10, D12, D9: LED, symbol Device:LED
- added D11: 1N4007, Diode_THT:D_DO-41_SOD81_P10.16mm_Horizontal, symbol Diode:1N4007
- added F1: Polyfuse_Small, symbol Device:Polyfuse_Small
- added J6: Screw_Terminal_01x03, symbol Connector:Screw_Terminal_01x03
- added J7: DS18s20, symbol Connector:Screw_Terminal_01x03
- added J8: DHT11, symbol Connector:Screw_Terminal_01x03
- added J9: Relay connector, symbol Connector:Screw_Terminal_01x06
- added R10, R11, R12, R9: R, symbol Device:R
- added SW1: SW_SPDT_312, symbol Switch:SW_SPDT_312
- added U10: TSR_1-2450, Converter_DCDC:Converter_DCDC_TRACO_TSR-1_THT, symbol Regulator_Switching:TSR_1-2450
Connections:
- net at U1.21 (GPIO15/JTAG): now also R9.1
- net at U1.23 (GPIO19): now also R11.2
- net at U1.25 (GPIO21): now also R10.2
- net +5V: now reaches U8.1 (VDD)
- net +5V: now also U6.3 (V_{DD}), U7.3 (V_{DD}), C2.1, R12.2, SW1.3 (A), U10.3 (Vout)
- net GND: now reaches U8.4 (GND)
- net GND: now also U6.1 (GND), U7.1 (GND), C1.2, C2.2, D12.1 (K), SW1.2 (C), U10.2 (GND)
- net Relay_Input1 renamed Relay_INPUT1
- net Relay_Input2 renamed Relay_INPUT2
- net Relay_Input4 renamed Relay_INPUT4
- new net: R9.2, SW1.1 (B)
- new net: D10.2 (A), R11.1
- new net: D9.2 (A), R10.1
- new net: D12.2 (A), R12.1
- new net: D11.1 (K), F1.1
- new net: C1.1, F1.2, U10.1 (Vin)
- new net +12V: D11.2 (A)
Other:
- moved on the sheet: U8
